Commit message: Initial commit: Base folder structure for Mobile Manipulators project

File: controllers/final_controller/Robot.urdf (robot description, URDF)
Before this commit: robot tiago, 61 links, 60 joints
Links:
- added link active_connector
Joints:
- added joint front_active_connector_joint: type fixed, parent front, child active_connector, origin xyz=0 0 -0.12 rpy=0 0 0
